File: axo.kicad_pcb (KiCad board)
At the start: 2 copper layers, 79.4 x 128.5 mm, 53 parts, among them Q1 MMBT3904, Q2 MMBT3904, Q3 MMBT3904, Q4 MMBT3904, U1 74HC02, U2 74HC00, U3 LM1117-5.0

Commit message: add readme
Parts:
- CON_A+1, CON_B+1: value Conn_01x06_Male -> Conn_01x06_Pin
- CON_A-1, CON_B-1: value Conn_01x06_Female -> Conn_01x06_Socket
- U4: renamed from U3; value LM1117-5.0 -> LM1117MP-5.0
- moved C1 1.93 mm to (172.6, 64.3), turned to 90 degrees
- moved R14 1.21 mm to (167.5, 117.8)
- moved R8 1.12 mm to (168.5, 57.5)
- moved R1 1.00 mm to (164.7, 57.5)
- moved Q4 0.95 mm to (167.4, 122.0), turned to 90 degrees
- moved Q2 0.93 mm to (168.4, 54.5), turned to 90 degrees
- moved R5 0.86 mm to (168.3, 51.5)
- moved D5 0.84 mm to (167.1, 127.0)
- moved R2 0.75 mm to (164.7, 51.5)
- moved R11 0.75 mm to (164.0, 130.2)
- moved Q1 0.69 mm to (164.6, 54.4), turned to -90 degrees
- moved R10 0.68 mm to (163.7, 125.0)
- moved R12 0.67 mm to (162.5, 117.8)
- moved D1 0.58 mm to (164.4, 49.5)
- moved R13 0.57 mm to (166.8, 125.0)
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- renumbered C3 to C1, C2 to C3, C1 to C4, C4 to C6, R12 to R11, R11 to R12, R18 to R13, R13 to R14, R17 to R16, R14 to R17, R16 to R18, R8 to R4, R7 to R5, R4 to R7, R5 to R8, U2 to U1, U1 to U3
Connections:
- CON_A-1 pad 6: GND -> GND2
- CON_B-1 pad 6: GND -> GND2
- D1 pad 1: Net-(D1-Pad1) -> Net-(D1-K)
- D2 pad 1: Net-(D2-Pad1) -> Net-(D2-K)
- D4 pad 1: Net-(D4-Pad1) -> Net-(D4-K)
- D5 pad 1: Net-(D5-Pad1) -> Net-(D5-K)
- IN_A1 pad S: GND -> GND2
- IN_A2 pad S: GND -> GND2
- IN_B1 pad S: GND -> GND2
- IN_B2 pad S: GND -> GND2
- OUT_A_AND1 pad S: GND -> GND2
- OUT_A_OR1 pad S: GND -> GND2
- OUT_A_XOR1 pad S: GND -> GND2
- OUT_B_AND1 pad S: GND -> GND2
- OUT_B_OR1 pad S: GND -> GND2
- OUT_B_XOR1 pad S: GND -> GND2
- Q1 pad 1: GND -> Net-(D1-K)
- Q1 pad 2: Net-(D1-Pad1) -> GND
- Q2 pad 1: GND -> Net-(D2-K)
- Q2 pad 2: Net-(D2-Pad1) -> GND
- Q3 pad 1: GND -> Net-(D4-K)
- Q3 pad 2: Net-(D4-Pad1) -> GND
- Q4 pad 1: GND -> Net-(D5-K)
- Q4 pad 2: Net-(D5-Pad1) -> GND
- R10 pad 1: Net-(D4-Pad1) -> Net-(D4-K)
- R11 pad 2: Net-(D4-Pad1) -> Net-(D4-K)
- R13 pad 1: Net-(D5-Pad1) -> Net-(D5-K)
- R17 pad 2: Net-(D5-Pad1) -> Net-(D5-K)
- R2 pad 1: Net-(D1-Pad1) -> Net-(D1-K)
- R3 pad 2: Net-(D1-Pad1) -> Net-(D1-K)
- R5 pad 1: Net-(D2-Pad1) -> Net-(D2-K)
- R9 pad 2: Net-(D2-Pad1) -> Net-(D2-K)
Routing:
- net Net-(D4-K): track 0.00 -> 8.61 mm
- net Net-(D5-Pad1): track 8.32 -> 0.00 mm
- net Net-(D2-K): track 0.00 -> 8.14 mm
- net Net-(D1-Pad1): track 7.25 -> 0.00 mm
- net Net-(D5-K): track 0.00 -> 6.80 mm
- net Net-(D4-Pad1): track 6.56 -> 0.00 mm
- net Net-(D1-K): track 0.00 -> 6.39 mm
- net Net-(D2-Pad1): track 5.43 -> 0.00 mm
- net Net-(R16-Pad1): track 55.2 -> 59.8 mm
- net Net-(R18-Pad1): track 70.2 -> 74.3 mm
- net GND: track 4.09 -> 0.00 mm
- net Net-(R6-Pad1): track 44.8 -> 48.2 mm
- net Net-(Q3-C): track 58.8 -> 61.6 mm
- net +5V: track 84.6 -> 86.5 mm
- net Net-(R7-Pad1): track 32.7 -> 34.2 mm
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- added copper zone on F.Cu, net GND2
Other:
- board size 79.4 x 128.5 mm -> 49.4 x 100 mm
- board text added: "REV 1.1"
- board text removed: "REV 1.0"
