File: axo_front.kicad_pcb (KiCad board)
At the start: 2 copper layers, 20 x 128.5 mm, 0 parts

Commit message: update pcb
Other:
- outline, holes or cut-outs redrawn
- board text removed: "AXOLOTL Front Panel - REV 1.0 Pierre Lamot 2024 JLCJLCJLCJLC"
