File: axo_middle.kicad_pcb (KiCad board)
At the start: 2 copper layers, 79.4 x 128.5 mm, 53 parts, among them Q1 MMBT3904, Q2 MMBT3904, Q3 MMBT3904, Q4 MMBT3904, U1 74HC02, U2 74HC00, U3 LM1117-5.0

Commit message: add readme
Parts:
- removed CON_A-1, CON_B-1: Conn_01x06_Female, Connector_PinSocket_2.54mm:PinSocket_1x06_P2.54mm_Vertical
- removed IN_A1, IN_A2, IN_B1, IN_B2, OUT_A_AND1, OUT_A_OR1, OUT_A_XOR1, OUT_B_AND1, OUT_B_OR1, OUT_B_XOR1: AudioJack2, Thonk:Jack_3.5mm_QingPu_WQP-PJ398SM_Vertical
- moved C1 1.93 mm to (172.6, 64.3), turned to 90 degrees
- moved R14 1.21 mm to (167.5, 117.8)
- moved R8 1.12 mm to (168.5, 57.5)
- moved R1 1.00 mm to (164.7, 57.5)
- moved Q4 0.95 mm to (167.4, 122.0), turned to 90 degrees
- moved Q2 0.93 mm to (168.4, 54.5), turned to 90 degrees
- moved R5 0.86 mm to (168.3, 51.5)
- moved D5 0.84 mm to (167.1, 127.0)
- moved R2 0.75 mm to (164.7, 51.5)
- moved R11 0.75 mm to (164.0, 130.2)
- moved Q1 0.69 mm to (164.6, 54.4), turned to -90 degrees
- moved R10 0.68 mm to (163.7, 125.0)
- moved R12 0.67 mm to (162.5, 117.8)
- moved D1 0.58 mm to (164.4, 49.5)
- moved R13 0.57 mm to (166.8, 125.0)
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- renumbered C3 to C1, C2 to C3, C1 to C4, C4 to C6, R12 to R11, R11 to R12, R18 to R13, R13 to R14, R17 to R16, R14 to R17, R16 to R18, R8 to R4, R7 to R5, R4 to R7, R5 to R8, U2 to U1, U1 to U3, U3 to U4
Connections:
- Q1 pad 1: GND -> Net-(D1-Pad1)
- Q1 pad 2: Net-(D1-Pad1) -> GND
- Q2 pad 1: GND -> Net-(D2-Pad1)
- Q2 pad 2: Net-(D2-Pad1) -> GND
- Q3 pad 1: GND -> Net-(D4-Pad1)
- Q3 pad 2: Net-(D4-Pad1) -> GND
- Q4 pad 1: GND -> Net-(D5-Pad1)
- Q4 pad 2: Net-(D5-Pad1) -> GND
Routing:
- net AO_TOP: track 46.4 -> 0.00 mm
- net B1_TOP: track 39.4 -> 0.00 mm
- net BA_TOP: track 37.3 -> 0.00 mm
- net AX_TOP: track 31.6 -> 0.00 mm
- net A2_TOP: track 29.5 -> 0.00 mm
- net B2_TOP: track 24.8 -> 0.00 mm
- net BX_TOP: track 21.0 -> 0.00 mm
- net AA_TOP: track 16.1 -> 0.00 mm
- net A1_TOP: track 13.2 -> 0.00 mm
- net BO_TOP: track 5.12 -> 0.00 mm
- net Net-(R16-Pad1): track 55.2 -> 59.8 mm
- net GND: track 4.09 -> 0.00 mm
- net Net-(R18-Pad1): track 70.2 -> 74.2 mm
- net Net-(R6-Pad1): track 44.8 -> 48.2 mm
- net Net-(R12-Pad2): track 58.8 -> 61.6 mm
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Other:
- board size 79.4 x 128.5 mm -> 19.4 x 100 mm
- board text added: "REV 1.1"
- board text removed: "AXOLOTL MIDDLE BOARD"
- board text removed: "REV 1.0"
